Commit message: 添加二阶摆实验，修复绘图bug

File: urdf/2_pendulum.urdf (robot description, URDF)
Before this commit: robot double_pendulum, 4 links, 3 joints
Links:
- removed link end_effector
- added link link_tcp, mass 0.2; collision sphere radius=0.04; visual sphere radius=0.04
Joints:
- joint second_to_end: child end_effector -> link_tcp
